Commit message: rm RoboschoolFork/tests/exponential_rewards/PPO2_1/events.out.tfevents.1573940334.gym

File: RoboschoolFork/roboschoolfork_nao/envs/models_robot/nao_description/urdf/naoV50_generated_urdf/nao.urdf (robot description, URDF)
Before this commit: robot NaoH25V50, 45 links, 44 joints
Links:
- link Head: geometry collision mesh filename=package://nao_meshes/meshes/HeadPitch_0.10.stl scale=0.1 0.1 0.1; visual mesh filename=package://nao_meshes/meshes/HeadPitch.1.dae scale=0.1 0.1 0.1
- link LAnklePitch: geometry collision mesh filename=package://nao_meshes/meshes/LAnklePitch_0.10.stl scale=0.1 0.1 0.1; visual mesh filename=package://nao_meshes/meshes/LAnklePitch.1.dae scale=0.1 0.1 0.1
- link LBicep: geometry collision mesh filename=package://nao_meshes/meshes/LShoulderRoll_0.10.stl scale=0.1 0.1 0.1; visual mesh filename=package://nao_meshes/meshes/LShoulderRoll.1.dae scale=0.1 0.1 0.1
- link LFinger11_link: geometry collision mesh filename=package://nao_meshes/meshes/LFinger11_0.10.stl scale=0.1 0.1 0.1; visual mesh filename=package://nao_meshes/meshes/LFinger11.1.dae scale=0.1 0.1 0.1
- link LFinger12_link: geometry collision mesh filename=package://nao_meshes/meshes/LFinger12_0.10.stl scale=0.1 0.1 0.1; visual mesh filename=package://nao_meshes/meshes/LFinger12.1.dae scale=0.1 0.1 0.1
- link LFinger13_link: geometry collision mesh filename=package://nao_meshes/meshes/LFinger13_0.10.stl scale=0.1 0.1 0.1; visual mesh filename=package://nao_meshes/meshes/LFinger13.1.dae scale=0.1 0.1 0.1
- link LFinger21_link: geometry collision mesh filename=package://nao_meshes/meshes/LFinger21_0.10.stl scale=0.1 0.1 0.1; visual mesh filename=package://nao_meshes/meshes/LFinger21.1.dae scale=0.1 0.1 0.1
- link LFinger22_link: geometry collision mesh filename=package://nao_meshes/meshes/LFinger22_0.10.stl scale=0.1 0.1 0.1; visual mesh filename=package://nao_meshes/meshes/LFinger22.1.dae scale=0.1 0.1 0.1
- link LFinger23_link: geometry collision mesh filename=package://nao_meshes/meshes/LFinger23_0.10.stl scale=0.1 0.1 0.1; visual mesh filename=package://nao_meshes/meshes/LFinger23.1.dae scale=0.1 0.1 0.1
- link LForeArm: geometry collision mesh filename=package://nao_meshes/meshes/LElbowRoll_0.10.stl scale=0.1 0.1 0.1; visual mesh filename=package://nao_meshes/meshes/LElbowRoll.1.dae scale=0.1 0.1 0.1
- link LHip: geometry collision mesh filename=package://nao_meshes/meshes/LHipRoll_0.10.stl scale=0.1 0.1 0.1; visual mesh filename=package://nao_meshes/meshes/LHipRoll.1.dae scale=0.1 0.1 0.1
- link LPelvis: geometry collision mesh filename=package://nao_meshes/meshes/LHipYawPitch_0.10.stl scale=0.1 0.1 0.1; visual mesh filename=package://nao_meshes/meshes/LHipYawPitch.1.dae scale=0.1 0.1 0.1
- link LShoulder: geometry collision mesh filename=package://nao_meshes/meshes/LShoulderPitch_0.10.stl scale=0.1 0.1 0.1; visual mesh filename=package://nao_meshes/meshes/LShoulderPitch.1.dae scale=0.1 0.1 0.1
- link LThigh: geometry collision mesh filename=package://nao_meshes/meshes/LHipPitch_0.10.stl scale=0.1 0.1 0.1; visual mesh filename=package://nao_meshes/meshes/LHipPitch.1.dae scale=0.1 0.1 0.1
- link LThumb1_link: geometry collision mesh filename=package://nao_meshes/meshes/LThumb1_0.10.stl scale=0.1 0.1 0.1; visual mesh filename=package://nao_meshes/meshes/LThumb1.1.dae scale=0.1 0.1 0.1
- link LThumb2_link: geometry collision mesh filename=package://nao_meshes/meshes/LThumb2_0.10.stl scale=0.1 0.1 0.1; visual mesh filename=package://nao_meshes/meshes/LThumb2.1.dae scale=0.1 0.1 0.1
- link LTibia: geometry collision mesh filename=package://nao_meshes/meshes/LKneePitch_0.10.stl scale=0.1 0.1 0.1; visual mesh filename=package://nao_meshes/meshes/LKneePitch.1.dae scale=0.1 0.1 0.1
- link Neck: geometry collision mesh filename=package://nao_meshes/meshes/HeadYaw_0.10.stl scale=0.1 0.1 0.1; visual mesh filename=package://nao_meshes/meshes/HeadYaw.1.dae scale=0.1 0.1 0.1
- link RAnklePitch: geometry collision mesh filename=package://nao_meshes/meshes/RAnklePitch_0.10.stl scale=0.1 0.1 0.1; visual mesh filename=package://nao_meshes/meshes/RAnklePitch.1.dae scale=0.1 0.1 0.1
- link RBicep: geometry collision mesh filename=package://nao_meshes/meshes/RShoulderRoll_0.10.stl scale=0.1 0.1 0.1; visual mesh filename=package://nao_meshes/meshes/RShoulderRoll.1.dae scale=0.1 0.1 0.1
- link RFinger11_link: geometry collision mesh filename=package://nao_meshes/meshes/RFinger11_0.10.stl scale=0.1 0.1 0.1; visual mesh filename=package://nao_meshes/meshes/RFinger11.1.dae scale=0.1 0.1 0.1
- link RFinger12_link: geometry collision mesh filename=package://nao_meshes/meshes/RFinger12_0.10.stl scale=0.1 0.1 0.1; visual mesh filename=package://nao_meshes/meshes/RFinger12.1.dae scale=0.1 0.1 0.1
- link RFinger13_link: geometry collision mesh filename=package://nao_meshes/meshes/RFinger13_0.10.stl scale=0.1 0.1 0.1; visual mesh filename=package://nao_meshes/meshes/RFinger13.1.dae scale=0.1 0.1 0.1
- link RFinger21_link: geometry collision mesh filename=package://nao_meshes/meshes/RFinger21_0.10.stl scale=0.1 0.1 0.1; visual mesh filename=package://nao_meshes/meshes/RFinger21.1.dae scale=0.1 0.1 0.1
- link RFinger22_link: geometry collision mesh filename=package://nao_meshes/meshes/RFinger22_0.10.stl scale=0.1 0.1 0.1; visual mesh filename=package://nao_meshes/meshes/RFinger22.1.dae scale=0.1 0.1 0.1
- link RFinger23_link: geometry collision mesh filename=package://nao_meshes/meshes/RFinger23_0.10.stl scale=0.1 0.1 0.1; visual mesh filename=package://nao_meshes/meshes/RFinger23.1.dae scale=0.1 0.1 0.1
- link RForeArm: geometry collision mesh filename=package://nao_meshes/meshes/RElbowRoll_0.10.stl scale=0.1 0.1 0.1; visual mesh filename=package://nao_meshes/meshes/RElbowRoll.1.dae scale=0.1 0.1 0.1
- link RHip: geometry collision mesh filename=package://nao_meshes/meshes/RHipRoll_0.10.stl scale=0.1 0.1 0.1; visual mesh filename=package://nao_meshes/meshes/RHipRoll.1.dae scale=0.1 0.1 0.1
- link RPelvis: geometry collision mesh filename=package://nao_meshes/meshes/RHipYawPitch_0.10.stl scale=0.1 0.1 0.1; visual mesh filename=package://nao_meshes/meshes/RHipYawPitch.1.dae scale=0.1 0.1 0.1
- link RShoulder: geometry collision mesh filename=package://nao_meshes/meshes/RShoulderPitch_0.10.stl scale=0.1 0.1 0.1; visual mesh filename=package://nao_meshes/meshes/RShoulderPitch.1.dae scale=0.1 0.1 0.1
- link RThigh: geometry collision mesh filename=package://nao_meshes/meshes/RHipPitch_0.10.stl scale=0.1 0.1 0.1; visual mesh filename=package://nao_meshes/meshes/RHipPitch.1.dae scale=0.1 0.1 0.1
- link RThumb1_link: geometry collision mesh filename=package://nao_meshes/meshes/RThumb1_0.10.stl scale=0.1 0.1 0.1; visual mesh filename=package://nao_meshes/meshes/RThumb1.1.dae scale=0.1 0.1 0.1
- link RThumb2_link: geometry collision mesh filename=package://nao_meshes/meshes/RThumb2_0.10.stl scale=0.1 0.1 0.1; visual mesh filename=package://nao_meshes/meshes/RThumb2.1.dae scale=0.1 0.1 0.1
- link RTibia: geometry collision mesh filename=package://nao_meshes/meshes/RKneePitch_0.10.stl scale=0.1 0.1 0.1; visual mesh filename=package://nao_meshes/meshes/RKneePitch.1.dae scale=0.1 0.1 0.1
- link l_ankle: geometry collision mesh filename=package://nao_meshes/meshes/LAnkleRoll_0.10.stl scale=0.1 0.1 0.1; visual mesh filename=package://nao_meshes/meshes/LAnkleRoll.1.dae scale=0.1 0.1 0.1
- link l_wrist: geometry collision mesh filename=package://nao_meshes/meshes/LWristYaw_0.10.stl scale=0.1 0.1 0.1; visual mesh filename=package://nao_meshes/meshes/LWristYaw.1.dae scale=0.1 0.1 0.1
- link r_ankle: geometry collision mesh filename=package://nao_meshes/meshes/RAnkleRoll_0.10.stl scale=0.1 0.1 0.1; visual mesh filename=package://nao_meshes/meshes/RAnkleRoll.1.dae scale=0.1 0.1 0.1
- link r_wrist: geometry collision mesh filename=package://nao_meshes/meshes/RWristYaw_0.10.stl scale=0.1 0.1 0.1; visual mesh filename=package://nao_meshes/meshes/RWristYaw.1.dae scale=0.1 0.1 0.1
- link torso: geometry collision mesh filename=package://nao_meshes/meshes/Torso_0.10.stl scale=0.1 0.1 0.1; visual mesh filename=package://nao_meshes/meshes/Torso.1.dae scale=0.1 0.1 0.1
